Commit message: ignition urdf edits

File: src/itls_robot_description/urdf/parts/itls_gazebo.xacro (robot description, xacro)
@@ -17,26 +17,6 @@
     <material>Gazebo/Black</material>
   </gazebo>
-  <!-- <gazebo reference="lidar_link">
+  <gazebo reference="lidar_front">
     <material>Gazebo/Black</material>
-  </gazebo> -->
-<!--WORKING DIFF DRIVE NO FRICTION FOR WHEELS REAR-->
-<!-- <gazebo>
-    <plugin name="diff_drive" filename="libgazebo_ros_diff_drive.so">
-      <ros>
-        <namespace>/</namespace>
-        <remapping>cmd_vel:=/cmd_vel</remapping>
-      </ros>
-      <left_joint>frontwhl_l_link</left_joint>
-      <right_joint>frontwhl_r_link</right_joint>
-      <wheel_separation>1.3005</wheel_separation>
-      <wheel_diameter>0.28</wheel_diameter>
-      <max_wheel_torque>20</max_wheel_torque>
-      <max_wheel_acceleration>1.0</max_wheel_acceleration>
-      <odometry_frame>odom</odometry_frame>
-      <robot_base_frame>base_link</robot_base_frame>
-      <publish_odom>true</publish_odom>
-      <publish_odom_tf>true</publish_odom_tf>
-      <publish_wheel_tf>true</publish_wheel_tf>
-    </plugin>
-  </gazebo>-->
+  </gazebo>
 </robot>

File: src/itls_robot_description/urdf/parts/itls_main.urdf.xacro (robot description, xacro)
@@ -6,5 +6,5 @@
   <xacro:include filename="itls_robot_base.xacro"/>
   <xacro:include filename="itls_robot_wheels.xacro"/>
-  <xacro:include filename="sensors.xacro"/>
-  <!-- <xacro:include filename="itls_gazebo.xacro"/> -->
+  <xacro:include filename="itls_scanners.xacro"/>
+  <xacro:include filename="itls_gazebo.xacro"/>
 </robot>

File: src/itls_robot_description/urdf/parts/itls_robot_base.xacro (robot description, xacro)
@@ -48,5 +48,5 @@
   <!-- Robot Footprint -->
   <link name="base_footprint"/>
-  <joint name="base_joint" type="fixed">
+  <joint name="base_link_T_base_footprint" type="fixed">
     <parent link="base_link"/>
     <child link="base_footprint"/>

File: src/itls_robot_description/urdf/parts/itls_robot_wheels.xacro (robot description, xacro)
@@ -9,5 +9,5 @@
   <xacro:property name="wheel_xoff" value="-0.16"/>
   <!-- keep in mind if there is problem in slippery between Gazebo and RVIZ
-  you can change the collision gemetry of the wheels into sphere without toaching the visuals
+  we can change the collision gemetry of the wheels into sphere without toaching the visuals
   Last time I checked the rotation it is pretty good no need -->
   <!-- Wheels Xacro and instances -->
@@ -31,5 +31,5 @@
       <xacro:cylinder_inertia m="50" r="${wheel_radius}" h="${wheel_width}"/>
     </link>
-    <joint name="${prefix}_joint" type="${fixedOrCont}">
+    <joint name="base_link_T_${prefix}" type="${fixedOrCont}">
       <parent link="base_link"/>
       <child link="${prefix}_link"/>
@@ -38,6 +38,6 @@
     </joint>
   </xacro:macro>
-  <xacro:wheel fixedOrCont="continuous" prefix="frontwhl_l" x_reflect="1" y_reflect="1" />
-  <xacro:wheel fixedOrCont="continuous" prefix="frontwhl_r" x_reflect="1" y_reflect="-1" />
+  <xacro:wheel fixedOrCont="fixed" prefix="frontwhl_l" x_reflect="1" y_reflect="1" />
+  <xacro:wheel fixedOrCont="fixed" prefix="frontwhl_r" x_reflect="1" y_reflect="-1" />
   <xacro:wheel fixedOrCont="continuous" prefix="rearwhl_l" x_reflect="-1" y_reflect="1" />
   <xacro:wheel fixedOrCont="continuous" prefix="rearwhl_r" x_reflect="-1" y_reflect="-1" />

File: src/itls_robot_description/urdf/parts/itls_scanners.xacro (robot description, xacro)
@@ -1,51 +1,53 @@
 <?xml version="1.0"?>
-<robot name="itls_robot" xmlns:xacro="http://www.ros.org/wiki/xacro">
+<robot name="itls_robot"
+  xmlns:xacro="http://www.ros.org/wiki/xacro">
   <!--Lidar Sensors Used for Gazebo-->
-  <link name="lidar_rear"/>
-  <joint name="base_link_to_lidar_rear" type="fixed">
-    <parent link="base_link"/>
-    <child link="lidar_rear"/>
-    <origin xyz="-1.28 -0.85 0.039" rpy="3.14159 0 2.53073"/> <!-- 180°, 0°, 145° in radians -->
-  </joint>
   <!-- Front LiDAR definition -->
-  <link name="lidar_front"/>
-  <joint name="base_link_to_lidar_front" type="fixed">
+  <joint name="base_link_T_lidar_front" type="fixed">
     <parent link="base_link"/>
     <child link="lidar_front"/>
-    <origin xyz="1.36 0.835 0.023" rpy="3.14159 0 -0.610865"/> <!-- 180°, 0°, -35° in radians -->
+    <origin xyz="1.36 0.835 0.023" rpy="3.14159 0 -0.610865"/>
   </joint>
-  <gazebo reference="scanner_front">
-   <sensor name="lidar" type="ray">
-    <always_on>true</always_on>
-    <visualize>true</visualize>
-    <update_rate>5</update_rate>
-    <ray>
-      <scan>
-        <horizontal>
-          <samples>360</samples>
-          <resolution>1.000000</resolution>
-          <min_angle>0.000000</min_angle>
-          <max_angle>5.10000</max_angle>
-        </horizontal>
-      </scan>
-      <range>
-        <min>0.120000</min>
-        <max>3.5</max>
-        <resolution>0.015000</resolution>
-      </range>
-      <noise>
-        <type>gaussian</type>
-        <mean>0.0</mean>
-        <stddev>0.01</stddev>
-      </noise>
-    </ray>
-    <plugin name="scan" filename="libgazebo_ros_ray_sensor.so">
-      <ros>
-        <remapping>~/out:=scan</remapping>
-      </ros>
-      <output_type>sensor_msgs/LaserScan</output_type>
-      <frame_name>lidar_link</frame_name>
-    </plugin>
-   </sensor>
+  <link name="lidar_front">
+    <visual>
+      <geometry>
+        <cylinder radius="0.05" length="0.05"/>
+      </geometry>
+    </visual>
+    <visual>
+      <origin xyz="0 0 -0.05"/>
+      <geometry>
+        <cylinder radius="0.01" length="0.1"/>
+      </geometry>
+    </visual>
+    <collision>
+      <geometry>
+        <cylinder radius="0.05" length="0.04"/>
+      </geometry>
+    </collision>
+    <xacro:cylinder_inertia m="2.0" r="0.05" h="0.04"/>
+  </link>
+  <gazebo reference="lidar_front">
+    <sensor name="scanner_front" type="gpu_lidar">
+      <pose> 0 0 0 0 0 0 </pose>
+      <topic>scan</topic>
+      <gz_frame_id>lidar_front</gz_frame_id>
+      <visualize>true</visualize>
+      <update_rate>10</update_rate>
+      <lidar>
+        <scan>
+          <horizontal>
+            <samples>360</samples>
+            <resolution>1</resolution>
+            <min_angle>-3.14</min_angle>
+            <max_angle>3.14</max_angle>
+          </horizontal>
+        </scan>
+        <range>
+          <min>0.3</min>
+          <max>12</max>
+        </range>
+      </lidar>
+    </sensor>
   </gazebo>
 </robot>
