Commit message: ignition edits and gazebo plugin calibrations

File: src/itls_robot_description/urdf/itls_robot_base.xacro (robot description, xacro)
@@ -4,5 +4,5 @@
   <xacro:property name="base_width" value="1.3005"/>
   <xacro:property name="base_length" value="4.136"/>
-  <xacro:property name="base_height" value="1.3"/>
+  <xacro:property name="base_height" value="0.5"/>
   <xacro:property name="base_link_to_front" value="2.3715"/>
   <xacro:property name="wheel_radius" value="0.14"/>
@@ -27,10 +27,10 @@
       </geometry>
     </collision>
-    <xacro:box_inertia m="1500" w="${base_width}" d="${base_length}" h="${base_height}"/>
+    <xacro:box_inertia m="10" w="${base_width}" d="${base_length}" h="${base_height}"/>
   </link>
   <joint name="base_link_T_robot_center" type="fixed">
     <parent link="base_link"/>
     <child link="robot_center"/>
-    <origin xyz="${base_link_to_lidar_rear + base_length_actual/2.0} 0.0 ${base_width/2.0}" rpy="0.0 0.0 0.0"/>
+    <origin xyz="${base_link_to_lidar_rear + base_length_actual/2.0} 0.0 ${base_height/2.0}" rpy="0.0 0.0 0.0"/>
   </joint>
   <link name="base_link_front"> </link>

File: src/itls_robot_description/urdf/itls_robot_wheels.xacro (robot description, xacro)
@@ -7,5 +7,5 @@
   <xacro:property name="wheel_ygap" value="0.07"/>
   <xacro:property name="wheel_zoff" value="0.0"/>
-  <xacro:property name="wheel_xoff" value="-0.16"/>
+  <xacro:property name="wheel_xoff" value="-0.5"/>
   <!-- keep in mind if there is problem in slippery between Gazebo and RVIZ
   we can change the collision gemetry of the wheels into sphere without toaching the visuals
@@ -29,5 +29,5 @@
         </geometry>
       </collision>
-      <xacro:cylinder_inertia m="50" r="${wheel_radius}" h="${wheel_width}"/>
+      <xacro:cylinder_inertia m="0.5" r="${wheel_radius}" h="${wheel_width}"/>
     </link>
     <joint name="base_link_T_${prefix}" type="${fixedOrCont}">
@@ -38,7 +38,33 @@
     </joint>
   </xacro:macro>
-  <xacro:wheel fixedOrCont="fixed" prefix="frontwhl_l" x_reflect="1" y_reflect="1" />
-  <xacro:wheel fixedOrCont="fixed" prefix="frontwhl_r" x_reflect="1" y_reflect="-1" />
+  <!-- <xacro:wheel fixedOrCont="continuous" prefix="frontwhl_l" x_reflect="1" y_reflect="1" /> -->
+  <!-- <xacro:wheel fixedOrCont="continuous" prefix="frontwhl_r" x_reflect="1" y_reflect="-1" /> -->
   <xacro:wheel fixedOrCont="continuous" prefix="rearwhl_l" x_reflect="-1" y_reflect="1" />
   <xacro:wheel fixedOrCont="continuous" prefix="rearwhl_r" x_reflect="-1" y_reflect="-1" />
+  <joint name="caster_wheel_joint" type="fixed">
+    <parent link="base_link"/>
+    <child link="caster_wheel"/>
+    <origin xyz="1.2 0 0"/>
+  </joint>
+  <link name="caster_wheel">
+    <visual>
+      <geometry>
+        <sphere radius="${wheel_radius}"/>
+      </geometry>
+      <material name="black"/>
+    </visual>
+    <collision>
+      <geometry>
+        <sphere radius="${wheel_radius}"/>
+      </geometry>
+    </collision>
+    <xacro:inertial_sphere mass="0.1" radius="${wheel_radius}">
+      <origin xyz="0 0 0" rpy="0 0 0"/>
+    </xacro:inertial_sphere>
+  </link>
+  <gazebo reference="caster_wheel">
+    <material>Gazebo/Black</material>
+    <mu1 value="0.001"/>
+    <mu2 value="0.001"/>
+  </gazebo>
 </robot>

File: src/itls_robot_description/urdf/itls_scanners.xacro (robot description, xacro)
@@ -14,9 +14,12 @@
         <cylinder radius="0.05" length="0.05"/>
       </geometry>
+      <material name="Red">
+        <color rgba="1.0 0 0 1.0"/>
+      </material>
     </visual>
     <visual>
       <origin xyz="0 0 -0.05"/>
       <geometry>
-        <cylinder radius="0.01" length="0.1"/>
+        <cylinder radius="0.05" length="0.05"/>
       </geometry>
     </visual>
@@ -26,11 +29,11 @@
       </geometry>
     </collision>
-    <xacro:cylinder_inertia m="2.0" r="0.05" h="0.04"/>
+    <xacro:cylinder_inertia m="0.002" r="0.05" h="0.04"/>
   </link>
   <gazebo reference="lidar_front">
-    <sensor name="scanner_front" type="gpu_lidar">
+    <sensor name="lidar_front" type="gpu_lidar">
       <pose> 0 0 0 0 0 0 </pose>
+      <ignition_frame_id>lidar_front</ignition_frame_id>
       <topic>scan</topic>
-      <gz_frame_id>lidar_front</gz_frame_id>
       <visualize>true</visualize>
       <update_rate>10</update_rate>
@@ -40,6 +43,6 @@
             <samples>360</samples>
             <resolution>1</resolution>
-            <min_angle>-3.14</min_angle>
-            <max_angle>3.14</max_angle>
+            <min_angle>2.7</min_angle>
+            <max_angle>7.1</max_angle>
           </horizontal>
         </scan>
