Commit message: add joint state publisher and tune gazebo motion

File: src/itls_robot_description/urdf/itls_gazebo.xacro (robot description, xacro)
@@ -14,5 +14,5 @@
       <max_linear_velocity>100</max_linear_velocity>
       <min_linear_velocity>-100</min_linear_velocity>
-      <!-- Input -->
+      <!-- Input Topic -->
       <topic>cmd_vel</topic>
       <!-- Output -->
@@ -27,4 +27,5 @@
       <joint_name>base_link_T_rearwhl_l</joint_name>
       <joint_name>base_link_T_rearwhl_r</joint_name>
+      <joint_name>caster_wheel_joint</joint_name>
     </plugin>
   </gazebo>

File: src/itls_robot_description/urdf/itls_robot_wheels.xacro (robot description, xacro)
@@ -8,7 +8,4 @@
   <xacro:property name="wheel_zoff" value="0.0"/>
   <xacro:property name="wheel_xoff" value="-0.5"/>
-  <!-- keep in mind if there is problem in slippery between Gazebo and RVIZ
-  we can change the collision gemetry of the wheels into sphere without toaching the visuals
-  Last time I checked the rotation it is pretty good no need -->
   <!-- Wheels Xacro and instances -->
   <xacro:macro name="wheel" params="prefix x_reflect y_reflect fixedOrCont">
@@ -42,5 +39,5 @@
   <xacro:wheel fixedOrCont="continuous" prefix="rearwhl_l" x_reflect="-1" y_reflect="1" />
   <xacro:wheel fixedOrCont="continuous" prefix="rearwhl_r" x_reflect="-1" y_reflect="-1" />
-  <joint name="caster_wheel_joint" type="fixed">
+  <joint name="caster_wheel_joint" type="continuous">
     <parent link="base_link"/>
     <child link="caster_wheel"/>
@@ -52,5 +49,7 @@
         <sphere radius="${wheel_radius}"/>
       </geometry>
-      <material name="black"/>
+      <material name="Black">
+        <color rgba="0 0 0 1"/>
+      </material>
     </visual>
     <collision>
@@ -63,8 +62,8 @@
     </xacro:inertial_sphere>
   </link>
-  <gazebo reference="caster_wheel">
+  <!-- <gazebo reference="caster_wheel">
     <material>Gazebo/Black</material>
-    <mu1 value="0.001"/>
-    <mu2 value="0.001"/>
-  </gazebo>
+    <mu1 value="0.1"/>
+    <mu2 value="0.1"/>
+  </gazebo> -->
 </robot>

Commit message: add lidar rear and some gazebo tunings

File: src/itls_robot_description/urdf/itls_gazebo.xacro (robot description, xacro)
@@ -7,5 +7,5 @@
       <left_joint>base_link_T_rearwhl_l</left_joint>
       <right_joint>base_link_T_rearwhl_r</right_joint>
-      <wheel_separation>1.3005</wheel_separation>
+      <wheel_separation>1.4505</wheel_separation>
       <wheel_radius>0.14</wheel_radius>
       <!-- Limits -->

File: src/itls_robot_description/urdf/itls_robot_base.xacro (robot description, xacro)
@@ -9,4 +9,5 @@
   <xacro:property name="base_length_actual" value="2.64"/>
   <xacro:property name="base_link_to_lidar_rear" value="-1.28"/>
+  <xacro:property name="base_mass" value="100"/>
   <!-- Robot Base -->
   <link name="base_link">
@@ -27,5 +28,5 @@
       </geometry>
     </collision>
-    <xacro:box_inertia m="10" w="${base_width}" d="${base_length}" h="${base_height}"/>
+    <xacro:box_inertia m="${base_mass}" w="${base_width}" d="${base_length}" h="${base_height}"/>
   </link>
   <joint name="base_link_T_robot_center" type="fixed">

File: src/itls_robot_description/urdf/itls_robot_wheels.xacro (robot description, xacro)
@@ -14,5 +14,5 @@
         <origin xyz="0 0 0" rpy="${pi/2} 0 0"/>
         <geometry>
-          <cylinder radius="${wheel_radius}" length="${wheel_width}"/>
+          <sphere radius="${wheel_radius}"/>
         </geometry>
         <material name="Black">
@@ -23,8 +23,10 @@
         <origin xyz="0 0 0" rpy="${pi/2} 0 0"/>
         <geometry>
-          <cylinder radius="${wheel_radius}" length="${wheel_width}"/>
+          <sphere radius="${wheel_radius}"/>
         </geometry>
       </collision>
-      <xacro:cylinder_inertia m="0.5" r="${wheel_radius}" h="${wheel_width}"/>
+      <xacro:inertial_sphere mass="4" radius="${wheel_radius}">
+        <origin xyz="0 0 0" rpy="0 0 0"/>
+      </xacro:inertial_sphere>
     </link>
     <joint name="base_link_T_${prefix}" type="${fixedOrCont}">
@@ -62,8 +64,8 @@
     </xacro:inertial_sphere>
   </link>
-  <!-- <gazebo reference="caster_wheel">
+  <gazebo reference="caster_wheel">
     <material>Gazebo/Black</material>
-    <mu1 value="0.1"/>
-    <mu2 value="0.1"/>
-  </gazebo> -->
+    <mu1 value="0.001"/>
+    <mu2 value="0.001"/>
+  </gazebo>
 </robot>

File: src/itls_robot_description/urdf/itls_scanners.xacro (robot description, xacro)
@@ -35,5 +35,56 @@
       <pose> 0 0 0 0 0 0 </pose>
       <ignition_frame_id>lidar_front</ignition_frame_id>
-      <topic>scan</topic>
+      <topic>scan_front</topic>
+      <visualize>true</visualize>
+      <update_rate>10</update_rate>
+      <lidar>
+        <scan>
+          <horizontal>
+            <samples>360</samples>
+            <resolution>1</resolution>
+            <min_angle>2.7</min_angle>
+            <max_angle>7.1</max_angle>
+          </horizontal>
+        </scan>
+        <range>
+          <min>0.3</min>
+          <max>12</max>
+        </range>
+      </lidar>
+    </sensor>
+  </gazebo>
+  <!-- Rear LiDAR definition -->
+  <joint name="base_link_T_lidar_rear" type="fixed">
+    <parent link="base_link"/>
+    <child link="lidar_rear"/>
+    <origin xyz="-1.28 -0.85 0.039" rpy="3.14159 0 2.530725"/>
+  </joint>
+  <link name="lidar_rear">
+    <visual>
+      <geometry>
+        <cylinder radius="0.05" length="0.05"/>
+      </geometry>
+      <material name="Red">
+        <color rgba="1.0 0 0 1.0"/>
+      </material>
+    </visual>
+    <visual>
+      <origin xyz="0 0 -0.05"/>
+      <geometry>
+        <cylinder radius="0.05" length="0.05"/>
+      </geometry>
+    </visual>
+    <collision>
+      <geometry>
+        <cylinder radius="0.05" length="0.04"/>
+      </geometry>
+    </collision>
+    <xacro:cylinder_inertia m="0.002" r="0.05" h="0.04"/>
+  </link>
+  <gazebo reference="lidar_rear">
+    <sensor name="lidar_rear" type="gpu_lidar">
+      <pose> 0 0 0 0 0 0 </pose>
+      <ignition_frame_id>lidar_rear</ignition_frame_id>
+      <topic>scan_rear</topic>
       <visualize>true</visualize>
       <update_rate>10</update_rate>
